File: MB-AIR-PIV/Main.sch (EAGLE design)
At the start: 25 parts, among them IC1 MEGA8-AI, IC2 LM1117DTX-5.0, J1 PIC_ICSP_MINI_5_PIN, J4 SPI, U4 LM1117 3.3, Y1 16MHZ

Commit message: new pwm
Parts:
- removed C3: 0.1uF, SparkFun-Passives:CAP0805
- removed C4: 22uF, adafruit:C-USC1206
- removed C5: 4.7uF, adafruit:C-USC1206
- removed J1: PIC_ICSP_MINI_5_PIN, SparkFun-Connectors:PIC_ICSP_MINI_5_PIN
- removed J2: (no value), SparkFun-Connectors:CONN_03JST-PTH-VERT
- removed J4: SPI, SparkFun-Connectors:AVR_SPI_PRG_6PTH
- removed U4: LM1117 3.3, SparkFun-PowerIC:V_REG_LM1117SOT223
- added BME280, OLED: (no value), SparkFun-Connectors:M04PTH
- added JP1: BT_RESET, SparkFun:M02PTH
- added SENSOR, VIN: (no value), SparkFun-Connectors:CONN_03JST-PTH-VERT
- added UPLOAD: PIC_ICSP_MINI_5_PIN, SparkFun-Connectors:PIC_ICSP_MINI_5_PIN
Connections:
- removed net 3.3V: C3.1, C4.1, U4.OUT, U4.OUT@1
- removed net SENS_IN: R13.2
- net 12V: now also R13.2, VIN.1; no longer J2.1
- net D3: now also VIN.2; no longer J2.2
- net D4: now also SENSOR.2
- net GND: now also BME280.2, JP1.2, OLED.2, SENSOR.3, UPLOAD.PGC, VIN.3; no longer C3.2, C4.2, C5.2, J1.PGC, J2.3, J4.6, U4.ADJ
- net MISO: no longer J4.1
- net MOSI: no longer J4.4
- net N$9: now also UPLOAD.VPP; no longer J1.VPP
- net RST: now also JP1.1; no longer J4.5
- net RXD: now also UPLOAD.GND; no longer J1.GND
- net SCK: no longer J4.3
- net SCL: now also BME280.3, OLED.3
- net SDA: now also BME280.4, OLED.4
- net TXD: now also UPLOAD.VCC; no longer J1.VCC
- net VCC: now also BME280.1, OLED.1, SENSOR.1, UPLOAD.PGD; no longer C5.1, J1.PGD, J4.2, U4.IN
Other:
- moved on the sheet: C10, C11, C12, C13, C14, C18, C6, C7, C8, D4, IC1, IC2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

Commit message: update
Parts:
- added X3: RELAY1, con-wago-500:W237-102
Connections:
- net 12V: now also X3-1.KL
- net GND: now also X3-2.KL
