File: MB-AIR-PIV/Main.brd (EAGLE design)
At the start: 160 x 100 mm, 25 parts, among them IC1 MEGA8-AI, IC2 LM1117DTX-5.0, J1 PIC_ICSP_MINI_5_PIN, J4 SPI, U4 LM1117 3.3, Y1 16MHZ

Commit message: new pwm
Parts:
- removed C3: 0.1uF, SparkFun-Passives:0805
- removed C4: 22uF, adafruit:C1206
- removed C5: 4.7uF, adafruit:C1206
- removed J1: PIC_ICSP_MINI_5_PIN, SparkFun-Connectors:PIC_ICSP_MINI_5_PIN
- removed J2: (no value), SparkFun-Connectors:JST-3-PTH-VERT
- removed J4: SPI, SparkFun-Connectors:2X3
- removed U4: LM1117 3.3, SparkFun-PowerIC:SOT223
- added BME280, OLED: (no value), SparkFun-Connectors:1X04
- added JP1: BT_RESET, SparkFun:1X02
- added SENSOR, VIN: (no value), SparkFun-Connectors:JST-3-PTH-VERT
- added UPLOAD: PIC_ICSP_MINI_5_PIN, SparkFun-Connectors:PIC_ICSP_MINI_5_PIN
- moved R15 94.5 mm to (12.7, 6.35), turned to 270 degrees
- moved C7 94.4 mm to (10.2, 25.4), turned to 270 degrees
- moved C11 92.9 mm to (40.6, 26.7)
- moved R13 91.2 mm to (15.2, 6.35), turned to 270 degrees
- moved R14 90.4 mm to (10.2, 6.35), turned to 90 degrees
- moved C6 89.2 mm to (7.62, 25.4), turned to 270 degrees
- moved Y1 84.4 mm to (8.89, 11.4), turned to 310 degrees
- moved D4 75.1 mm to (18.3, 7.62), turned to 270 degrees
- moved C18 70.6 mm to (12.7, 25.4), turned to 90 degrees
- moved C10 69.7 mm to (39.4, 7.62)
- moved C14 67.6 mm to (15.2, 25.4), turned to 90 degrees
- moved C13 66.9 mm to (17.8, 25.4), turned to 90 degrees
- moved C12 66.2 mm to (20.3, 25.4), turned to 90 degrees
- moved C8 62.0 mm to (7.62, 6.35), turned to 90 degrees
- moved R9 61.5 mm to (7.62, 29.2), turned to 180 degrees
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Connections:
- removed net 3.3V: C3.1, C4.1, U4.2, U4.4
- removed net SENS_IN: R13.2
- net 12V: now also R13.2, VIN.1; no longer J2.1
- net D3: now also VIN.2; no longer J2.2
- net D4: now also SENSOR.2
- net GND: now also BME280.2, JP1.2, OLED.2, SENSOR.3, UPLOAD.5, VIN.3; no longer C3.2, C4.2, C5.2, J1.5, J2.3, J4.6, U4.1
- net MISO: no longer J4.1
- net MOSI: no longer J4.4
- net N$9: now also UPLOAD.1; no longer J1.1
- net RST: now also JP1.1; no longer J4.5
- net RXD: now also UPLOAD.3; no longer J1.3
- net SCK: no longer J4.3
- net SCL: now also BME280.3, OLED.3
- net SDA: now also BME280.4, OLED.4
- net TXD: now also UPLOAD.2; no longer J1.2
- net VCC: now also BME280.1, OLED.1, SENSOR.1, UPLOAD.4; no longer C5.1, J1.4, J4.2, U4.3
Other:
- board size 160 x 100 mm -> 50.8 x 32.7 mm

Commit message: update
Parts:
- added X3: RELAY1, con-wago-500:W237-102
- moved C8 20.7 mm to (11.4, 26.7)
- moved JP1 17.0 mm to (10.2, 21.6), turned to 270 degrees
- moved R13 13.0 mm to (27.9, 8.89)
- moved R15 11.7 mm to (24.1, 8.89)
- moved BME280 11.5 mm to (21.6, 3.81)
- moved C7 11.5 mm to (21.6, 26.7)
- moved R14 10.5 mm to (20.3, 8.89)
- moved UPLOAD 10.2 mm to (6.35, 3.81), turned to 0 degrees
- moved IC2 9.25 mm to (30.5, 20.3), turned to 0 degrees
- moved D4 9.01 mm to (26.7, 4.32), turned to 0 degrees
- moved C12 6.48 mm to (26.7, 26.7)
- moved C18 6.48 mm to (19.1, 26.7)
- moved C6 6.48 mm to (14.0, 26.7)
- moved C13 6.48 mm to (24.1, 26.7)
- moved OLED 5.24 mm to (16.5, 30.5)
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Connections:
- net 12V: now also X3.1
- net GND: now also X3.2
Routing:
- net GND: track 0.00 -> 251.6 mm
- net VCC: track 0.00 -> 206.6 mm
- net 12V: track 0.00 -> 140.1 mm
- net SCL: track 0.00 -> 51.7 mm
- net N$12: track 0.00 -> 50.4 mm
- net SDA: track 0.00 -> 44.9 mm
- net A0: track 0.00 -> 31.6 mm
- net N$9: track 0.00 -> 31.5 mm
- net RXD: track 0.00 -> 25.4 mm
- net TXD: track 0.00 -> 21.7 mm, vias 0 -> 2
- net RST: track 0.00 -> 16.6 mm
- net D4: track 0.00 -> 14.0 mm
- net D3: track 0.00 -> 10.7 mm
- net N$8: track 0.00 -> 6.33 mm
- net N$7: track 0.00 -> 4.61 mm
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- added copper zone on layer 16, net B
- added copper zone on layer 1, net T
Other:
- board size 50.8 x 32.7 mm -> 44.5 x 34.3 mm

Commit message: update
Parts:
- moved R9 4.20 mm to (11.9, 26.7), turned to 90 degrees
- moved C8 1.78 mm to (9.65, 26.7), turned to 270 degrees
- moved R13 1.27 mm to (27.9, 7.62), turned to 0 degrees
- moved R14 1.27 mm to (20.3, 7.62), turned to 0 degrees
- moved R15 1.27 mm to (24.1, 7.62), turned to 0 degrees
- moved C6 0.25 mm to (14.2, 26.7), turned to 90 degrees
- turned C14 to 270 degrees
- turned IC1 to 45 degrees
- turned Y1 to 314 degrees
Routing:
- net GND: track 251.6 -> 201.7 mm, vias 0 -> 4
- net VCC: track 206.6 -> 171.3 mm, vias 0 -> 5
- net N$12: track 50.4 -> 42.5 mm, vias 0 -> 2
- net 12V: track 140.1 -> 147.7 mm
- net SDA: track 44.9 -> 51.8 mm
- net TXD: track 21.7 -> 26.5 mm
- net RST: track 16.6 -> 12.6 mm
- net SCL: track 51.7 -> 48.6 mm, vias 0 -> 2
- net D3: track 10.7 -> 13.5 mm
- net N$9: track 31.5 -> 29.8 mm
- net D4: track 14.0 -> 15.5 mm
- net A0: track 31.6 -> 30.4 mm
- net RXD: track 25.4 -> 26.2 mm, vias 0 -> 2
- net N$7: track 4.61 -> 5.39 mm
- net N$5: track 3.21 -> 3.92 mm
