File: ECU-V3/Main.sch (EAGLE design)
At the start: 54 parts, among them IC1 MEGA8-AI, IC2 LM1117DTX-5.0, Q3 BSS138BK, Q4 BSS138BK, T3 BC817, U1 MCP4922-E/SL, U2 HM-11, U4 LM1117 3.3, Y1 16MHZ

Commit message: update
Connections:
- removed net N$9: ECU.5, SENSOR.5
- net GND: now also ECU.5, SENSOR.5
Changed lines of the file:
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@@
 <label x="198.12" y="-2.54" size="1.778" layer="95"/>
+</segment>
+<segment>
+<pinref part="ECU" gate="G$1" pin="5"/>
+<wire x1="261.62" y1="121.92" x2="256.54" y2="121.92" width="0.1524" layer="91"/>
+<wire x1="256.54" y1="121.92" x2="256.54" y2="142.24" width="0.1524" layer="91"/>
+<pinref part="SENSOR" gate="G$1" pin="5"/>
+<wire x1="256.54" y1="142.24" x2="261.62" y2="142.24" width="0.1524" layer="91"/>
+<label x="243.84" y="121.92" size="1.778" layer="95"/>
+<label x="243.84" y="142.24" size="1.778" layer="95"/>
 </segment>
 </net>
@@
 <pinref part="SENSOR" gate="G$1" pin="3"/>
 <wire x1="261.62" y1="147.32" x2="243.84" y2="147.32" width="0.1524" layer="91"/>
-<label x="241.3" y="147.32" size="1.778" layer="95"/>
+<label x="243.84" y="147.32" size="1.778" layer="95"/>
 </segment>
 </net>
@@
 <wire x1="254" y1="152.4" x2="261.62" y2="152.4" width="0.1524" layer="91"/>
 <label x="243.84" y="132.08" size="1.778" layer="95"/>
+<label x="243.84" y="152.4" size="1.778" layer="95"/>
 </segment>
 </net>
@@
 </segment>
 </net>
-<net name="N$9" class="0">
-<segment>
-<pinref part="ECU" gate="G$1" pin="5"/>
-<wire x1="261.62" y1="121.92" x2="256.54" y2="121.92" width="0.1524" layer="91"/>
-<wire x1="256.54" y1="121.92" x2="256.54" y2="142.24" width="0.1524" layer="91"/>
-<pinref part="SENSOR" gate="G$1" pin="5"/>
-<wire x1="256.54" y1="142.24" x2="261.62" y2="142.24" width="0.1524" layer="91"/>
-</segment>
-</net>
