File: ECU-V4/Main.brd (EAGLE design)
At the start: 85.1 x 100 mm, 54 parts, among them IC1 MEGA8-AI, IC2 LM1117DTX-5.0, Q3 BSS138BK, Q4 BSS138BK, T3 BC817, U1 MCP4922-E/SL, U2 HM-11, U4 LM1117 3.3, Y1 16MHZ

Commit message: update
Parts:
- added C15: 10uf, adafruit:153CLV-0605
- added C16: 0.1, SparkFun-Passives:CAP-PTH-5MM
- added D3: SZ105B, diode:DO-214AC
- added R19, R8: 10k, SparkFun-Resistors:0805
- added R20: 20k, SparkFun-Resistors:0805
- added U$1: MCP3424-E/SL, Microchip_By_element14_Batch_1:SOIC127P600X175-14N
- moved R12 83.5 mm to (39.4, 7.62), turned to 90 degrees
- moved R17 82.8 mm to (41.9, 7.62), turned to 270 degrees
- moved R18 82.5 mm to (44.5, 7.62), turned to 90 degrees
- moved Y1 72.7 mm to (25.4, 12.7), turned to 315 degrees
- moved D4 72.5 mm to (110.5, 44.5)
- moved C13 72.2 mm to (22.9, 15.2), turned to 315 degrees
- moved C6 63.7 mm to (34.3, 22.9), turned to 315 degrees
- moved C7 63.1 mm to (35.6, 24.1), turned to 315 degrees
- moved JP2 62.5 mm to (24.1, 7.62)
- moved R7 62.1 mm to (67.3, 49.5), turned to 270 degrees
- moved C8 59.7 mm to (22.9, 26.7), turned to 270 degrees
- moved IC2 59.2 mm to (74.9, 72.4), turned to 90 degrees
- moved R9 56.7 mm to (25.4, 26.7), turned to 90 degrees
- moved T3 53.4 mm to (48.3, 7.62), turned to 270 degrees
- moved U2 53.4 mm to (57.1, 54.6), flipped to the bottom, turned to 0 degrees
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Connections:
- net 14 renamed OUTSIGN
- net SE renamed SENSOROUTTEMP
- net SS renamed SENSORINTEMP
- new net GNDAIR: D3.A, ECU.2, R20.1, SENSOR.2, U$1.2
- new net GNDTEMP: ECU.5, SENSOR.5
- net GND: now also C15.-, C16.2, U$1.10, U$1.5, U$1.9; no longer ECU.2, ECU.5, SENSOR.2, SENSOR.5
- net SCL: now also R19.2, U$1.8
- net SDA: now also R8.1, U$1.7
- net SENS_IN: now also D3.C, R20.2, U$1.1
- net VCC: now also C15.+, C16.1, R19.1, R8.2, U$1.6
Other:
- board size 85.1 x 100 mm -> 110.5 x 83.8 mm

Commit message: update
Parts:
- removed C16: 0.1, SparkFun-Passives:CAP-PTH-5MM
- removed D4: SZ105B, diode:DO-214AC
- added C17: 0.1uF, SparkFun-Passives:0805
- added D5: 4148, semicon-smd-ipc:SOD80
- D3: value SZ105B -> 4148; device diode:DO-214AC -> semicon-smd-ipc:SOD80
- LED1: value BT_STATE -> BT
- moved D3 103.5 mm to (16.8, 23.2), turned to 270 degrees
- moved C11 75.8 mm to (21.6, 44.5), turned to 270 degrees
- moved C10 75.4 mm to (11.4, 43.2)
- moved IC2 74.7 mm to (11.4, 33.0)
- moved U4 72.8 mm to (21.6, 34.3)
- moved R19 66.1 mm to (47.8, 20.3), turned to 90 degrees
- moved C15 61.0 mm to (29.2, 44.5), turned to 270 degrees
- moved C1 57.7 mm to (31.8, 24.1)
- moved R2 55.8 mm to (36.8, 26.7), turned to 90 degrees
- moved R15 53.6 mm to (22.9, 16.5), turned to 90 degrees
- moved R13 52.6 mm to (25.4, 16.5), turned to 270 degrees
- moved R5 52.1 mm to (25.4, 27.9), turned to 270 degrees
- moved R16 51.8 mm to (50.8, 41.9), turned to 90 degrees
- moved Q4 51.2 mm to (44.5, 26.7), turned to 270 degrees
- moved D1 51.2 mm to (47.8, 26.7), turned to 90 degrees
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Connections:
- net A0: now also D3.1; no longer D4.C
- net GND: now also C17.2, D3.2; no longer C16.2, D4.A
- net GNDAIR: now also D5.2; no longer D3.A
- net SENS_IN: now also D5.1; no longer D3.C
- net VCC: now also C17.1; no longer C16.1
Routing:
- net GND: track 0.00 -> 339.6 mm, vias 0 -> 5
- net VCC: track 0.00 -> 242.1 mm, vias 0 -> 7
- net A1: track 0.00 -> 99.1 mm, vias 0 -> 3
- net 12V: track 0.00 -> 83.2 mm, vias 0 -> 2
- net GNDAIR: track 0.00 -> 72.8 mm, vias 0 -> 4
- net 3.3V: track 0.00 -> 67.7 mm, vias 0 -> 2
- net SENS_IN: track 0.00 -> 57.0 mm, vias 0 -> 4
- net N$31: track 0.00 -> 56.8 mm, vias 0 -> 1
- net D9: track 0.00 -> 53.8 mm, vias 0 -> 2
- net SENSOROUTTEMP: track 0.00 -> 53.5 mm, vias 0 -> 1
- net GNDTEMP: track 0.00 -> 52.4 mm
- net D8: track 0.00 -> 46.2 mm, vias 0 -> 2
- net SCL: track 0.00 -> 44.3 mm, vias 0 -> 2
- net SDA: track 0.00 -> 40.1 mm, vias 0 -> 2
- net N$1: track 0.00 -> 35.8 mm, vias 0 -> 1
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Other:
- board size 110.5 x 83.8 mm -> 55.9 x 49.5 mm
