File: ECU-V4/Main.sch (EAGLE design)
At the start: 58 parts, among them IC1 MEGA8-AI, IC2 LM1117DTX-5.0, J6 Remote, J7 AVR_SPI_PROG_3X2TESTPOINTS, Q3 BSS138BK, Q4 BSS138BK, T3 BC817, U1 MCP4922-E/SL, U2 HM-11, U4 LM1117 3.3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

Commit message: update
Parts:
- removed J5: (no value), SparkFun-Connectors:CONN_04JST-PTH
- removed J6: Remote, SparkFun-Connectors:CONN_04JST-PTH
- removed J7: AVR_SPI_PROG_3X2TESTPOINTS, SparkFun-Connectors:AVR_SPI_PROG_3X2TESTPOINTS
- removed JP3, JP4: (no value), SparkFun:M05PTH
- added C16: 0.1, SparkFun-Passives:CAPPTH1
- added C8: 0.1uF, SparkFun-Passives:CAP0805
- added D3: SZ105B, diode:DIODE-DO-214AC
- added ECU, SENSOR: (no value), SparkFun:M05PTH
- added R19: 10k, SparkFun-Resistors:RESISTOR0805-RES
- added R20: 20k, SparkFun-Resistors:RESISTOR0805-RES
- added U$1: MCP3424-E/SL, Microchip_By_element14_Batch_1:MCP3424-E/SL
- C15: value 0.1uF -> 10uf; device SparkFun-Passives:CAP0805 -> adafruit:CPOL-US153CLV-0605
- JP1: value BT_RESET -> (none); device SparkFun:M02PTH -> SparkFun:M07
- JP2: value BT_KEY -> (none); device SparkFun:M02PTH -> SparkFun:M05PTH
Connections:
- removed net 14: JP4.3, U1.VOUTA
- removed net N$18: C15.1, J7.1
- removed net N$4: JP1.1, R8.2, U2.RESETB
- removed net N$9: JP3.5, JP4.5
- removed net SE: JP4.4, U$10.SWCOMMON
- removed net SS: JP3.4, U$10.SWCLOSE
- new net GNDAIR: D3.A, ECU.2, R20.1, SENSOR.2, U$1.CH1-
- new net GNDTEMP: ECU.5, SENSOR.5
- new net N$10: C8.1, JP2.1
- new net OUTSIGN: ECU.3, U1.VOUTA
- new net SENSORINTEMP: SENSOR.4, U$10.SWCLOSE
- new net SENSOROUTTEMP: ECU.4, U$10.SWCOMMON
- net 12V: now also ECU.1, SENSOR.1; no longer JP3.1, JP4.1
- net 3.3V: no longer R8.1
- net A2: now also JP1.3; no longer J5.2
- net A3: now also JP1.4; no longer J5.1
- net D2: now also JP1.5; no longer J6.4
- net D3: now also JP1.6; no longer J6.3
- net D4: now also JP1.7; no longer J6.2
- net GND: now also C15.-, C16.2, JP2.4, U$1.ADR0, U$1.ADR1, U$1.VSS; no longer J5.3, J7.5, JP2.2, JP3.2, JP4.2
- net N$2: no longer JP2.1
- net RST: now also C8.2; no longer C15.2
- net RXD: now also JP2.2; no longer J7.3
- net SCL: now also R19.2, U$1.SCL
- net SDA: now also R8.1, U$1.SDA
- net SENS_IN: now also D3.C, R20.2, SENSOR.3, U$1.CH1+; no longer JP3.3
- net TXD: now also JP2.3; no longer J7.2
- net VCC: now also C15.+, C16.1, JP1.1, JP2.5, R19.1, R8.2, U$1.VDD; no longer J5.4, J7.4
Other:
- moved on the sheet: C1, C10, C11, C12, C13, C14, C18, C2, C3, C4, C5, C6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

Commit message: update
Parts:
- removed C16: 0.1, SparkFun-Passives:CAPPTH1
- removed D4: SZ105B, diode:DIODE-DO-214AC
- added C17: 0.1uF, SparkFun-Passives:CAP0805
- added D5: 4148, semicon-smd-ipc:D-SOD-80
- D3: value SZ105B -> 4148; device diode:DIODE-DO-214AC -> semicon-smd-ipc:D-SOD-80
- LED1: value BT_STATE -> BT
Connections:
- net A0: now also D3.C; no longer D4.C
- net GND: now also C17.2, D3.A; no longer C16.2, D4.A
- net GNDAIR: now also D5.A; no longer D3.A
- net SENS_IN: now also D5.C; no longer D3.C
- net VCC: now also C17.1; no longer C16.1
Other:
- moved on the sheet: D3
Changed lines of the file:
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@@
 <part name="R16" library="SparkFun-Resistors" deviceset="RESISTOR" device="0805-RES" value="1k"/>
 <part name="LED3" library="adafruit" deviceset="LED" device="3MM" value="RY"/>
-<part name="LED1" library="adafruit" deviceset="LED" device="3MM" value="BT_STATE"/>
+<part name="LED1" library="adafruit" deviceset="LED" device="3MM" value="BT"/>
 <part name="LED2" library="adafruit" deviceset="LED" device="3MM" value="PW"/>
 <part name="GND12" library="SparkFun-Aesthetics" deviceset="GND" device=""/>
@@
 <part name="C12" library="SparkFun-Passives" deviceset="CAP" device="0805" value="0.1uF"/>
 <part name="C10" library="adafruit" deviceset="CPOL-US" device="153CLV-1010" value="220/50"/>
-<part name="D4" library="diode" deviceset="DIODE-" device="DO-214AC" value="SZ105B"/>
 <part name="C18" library="SparkFun-Passives" deviceset="CAP" device="0805" value="0.1"/>
 <part name="C13" library="SparkFun-Passives" deviceset="CAP" device="0805" value="0.1uF"/>
@@
 <part name="C8" library="SparkFun-Passives" deviceset="CAP" device="0805" value="0.1uF"/>
 <part name="U$1" library="Microchip_By_element14_Batch_1" deviceset="MCP3424-E/SL" device=""/>
-<part name="C16" library="SparkFun-Passives" deviceset="CAP" device="PTH1" value="0.1"/>
 <part name="SUPPLY7" library="SparkFun-Aesthetics" deviceset="VCC" device=""/>
 <part name="GND5" library="SparkFun" deviceset="GND" device=""/>
@@
 <part name="R20" library="SparkFun-Resistors" deviceset="RESISTOR" device="0805-RES" value="20k"/>
 <part name="GND11" library="SparkFun" deviceset="GND" device=""/>
-<part name="D3" library="diode" deviceset="DIODE-" device="DO-214AC" value="SZ105B"/>
 <part name="C15" library="adafruit" deviceset="CPOL-US" device="153CLV-0605" value="10uf"/>
+<part name="C17" library="SparkFun-Passives" deviceset="CAP" device="0805" value="0.1uF"/>
+<part name="D5" library="semicon-smd-ipc" library_urn="urn:adsk.eagle:library:353" deviceset="D-" device="SOD-80" package3d_urn="urn:adsk.eagle:package:26309/1" value="4148"/>
+<part name="D3" library="semicon-smd-ipc" library_urn="urn:adsk.eagle:library:353" deviceset="D-" device="SOD-80" package3d_urn="urn:adsk.eagle:package:26309/1" value="4148"/>
 </parts>
 <sheets>
@@
 <attribute name="VALUE" x="8.636" y="66.929" size="1.778" layer="96"/>
 </instance>
-<instance part="D4" gate="G$1" x="276.86" y="30.48" smashed="yes" rot="R90">
-<attribute name="NAME" x="276.3774" y="40.64" size="1.778" layer="95" rot="R90"/>
-<attribute name="VALUE" x="279.1714" y="40.64" size="1.778" layer="96" rot="R90"/>
-</instance>
 <instance part="C18" gate="G$1" x="269.24" y="27.94" smashed="yes">
 <attribute name="NAME" x="270.764" y="30.861" size="1.778" layer="95"/>
@@
 <attribute name="VALUE" x="162.1282" y="105.1306" size="2.0828" layer="96" ratio="10" rot="SR0"/>
 </instance>
-<instance part="C16" gate="G$1" x="132.08" y="116.84" smashed="yes">
-<attribute name="NAME" x="133.604" y="119.761" size="1.778" layer="95"/>
-<attribute name="VALUE" x="133.604" y="114.681" size="1.778" layer="96"/>
-</instance>
 <instance part="SUPPLY7" gate="G$1" x="121.92" y="160.02" smashed="yes">
 <attribute name="VALUE" x="120.904" y="163.576" size="1.778" layer="96"/>
@@
 <attribute name="VALUE" x="139.7" y="134.62" size="1.778" layer="96"/>
 </instance>
-<instance part="D3" gate="G$1" x="137.16" y="147.32" smashed="yes" rot="R90">
-<attribute name="NAME" x="136.6774" y="157.48" size="1.778" layer="95" rot="R90"/>
-<attribute name="VALUE" x="139.4714" y="157.48" size="1.778" layer="96" rot="R90"/>
-</instance>
 <instance part="C15" gate="G$1" x="124.46" y="119.38" smashed="yes">
 <attribute name="NAME" x="125.476" y="120.015" size="1.778" layer="95"/>
 <attribute name="VALUE" x="125.476" y="115.189" size="1.778" layer="96"/>
+</instance>
+<instance part="C17" gate="G$1" x="132.08" y="116.84" smashed="yes">
+<attribute name="NAME" x="133.604" y="119.761" size="1.778" layer="95"/>
+<attribute name="VALUE" x="133.604" y="114.681" size="1.778" layer="96"/>
+</instance>
+<instance part="D5" gate="G$1" x="137.16" y="147.32" smashed="yes" rot="R90">
+<attribute name="NAME" x="135.382" y="144.78" size="1.778" layer="95" rot="R90"/>
+<attribute name="VALUE" x="140.843" y="144.78" size="1.778" layer="96" rot="R90"/>
+</instance>
+<instance part="D3" gate="G$1" x="276.86" y="30.48" smashed="yes" rot="R90">
+<attribute name="NAME" x="275.082" y="27.94" size="1.778" layer="95" rot="R90"/>
+<attribute name="VALUE" x="280.543" y="27.94" size="1.778" layer="96" rot="R90"/>
 </instance>
 </instances>
@@
 <pinref part="GND10" gate="1" pin="GND"/>
 <wire x1="284.48" y1="22.86" x2="284.48" y2="20.32" width="0.1524" layer="91"/>
-<pinref part="D4" gate="G$1" pin="A"/>
 <wire x1="276.86" y1="27.94" x2="276.86" y2="22.86" width="0.1524" layer="91"/>
 <wire x1="276.86" y1="22.86" x2="284.48" y2="22.86" width="0.1524" layer="91"/>
@@
 <wire x1="269.24" y1="22.86" x2="276.86" y2="22.86" width="0.1524" layer="91"/>
 <junction x="276.86" y="22.86"/>
+<pinref part="D3" gate="G$1" pin="A"/>
 </segment>
 <segment>
@@
 <pinref part="GND5" gate="1" pin="GND"/>
 <wire x1="119.38" y1="109.22" x2="119.38" y2="111.76" width="0.1524" layer="91"/>
-<pinref part="C16" gate="G$1" pin="2"/>
 <wire x1="132.08" y1="114.3" x2="132.08" y2="111.76" width="0.1524" layer="91"/>
 <wire x1="132.08" y1="111.76" x2="124.46" y2="111.76" width="0.1524" layer="91"/>
@@
 <junction x="124.46" y="111.76"/>
 <pinref part="C15" gate="G$1" pin="-"/>
+<pinref part="C17" gate="G$1" pin="2"/>
 </segment>
 <segment>
@@
 <pinref part="SUPPLY7" gate="G$1" pin="VCC"/>
 <wire x1="121.92" y1="154.94" x2="121.92" y2="160.02" width="0.1524" layer="91"/>
-<pinref part="C16" gate="G$1" pin="1"/>
 <wire x1="121.92" y1="154.94" x2="132.08" y2="154.94" width="0.1524" layer="91"/>
 <wire x1="132.08" y1="154.94" x2="132.08" y2="127" width="0.1524" layer="91"/>
@@
 <pinref part="R19" gate="G$1" pin="1"/>
 <pinref part="C15" gate="G$1" pin="+"/>
+<pinref part="C17" gate="G$1" pin="1"/>
 </segment>
 </net>
@@
 <wire x1="266.7" y1="35.56" x2="269.24" y2="35.56" width="0.1524" layer="91"/>
 <junction x="284.48" y="35.56"/>
-<pinref part="D4" gate="G$1" pin="C"/>
 <wire x1="269.24" y1="35.56" x2="276.86" y2="35.56" width="0.1524" layer="91"/>
 <wire x1="276.86" y1="35.56" x2="284.48" y2="35.56" width="0.1524" layer="91"/>
@@
 <wire x1="269.24" y1="33.02" x2="269.24" y2="35.56" width="0.1524" layer="91"/>
 <junction x="269.24" y="35.56"/>
+<pinref part="D3" gate="G$1" pin="C"/>
 </segment>
 </net>
@@
 <junction x="142.24" y="152.4"/>
 <label x="119.38" y="152.4" size="1.778" layer="95"/>
-<pinref part="D3" gate="G$1" pin="C"/>
 <wire x1="137.16" y1="149.86" x2="137.16" y2="152.4" width="0.1524" layer="91"/>
 <junction x="137.16" y="152.4"/>
+<pinref part="D5" gate="G$1" pin="C"/>
 </segment>
 </net>
@@
 <wire x1="147.32" y1="142.24" x2="142.24" y2="142.24" width="0.1524" layer="91"/>
 <label x="119.38" y="142.24" size="1.778" layer="95"/>
-<pinref part="D3" gate="G$1" pin="A"/>
 <wire x1="137.16" y1="142.24" x2="137.16" y2="144.78" width="0.1524" layer="91"/>
 <junction x="137.16" y="142.24"/>
-</segment>
-</net>
+<pinref part="D5" gate="G$1" pin="A"/>
+</segment>
+</net>
