File: MB_AutoCar/main.brd (EAGLE design)
At the start: 210.8 x 146.1 mm, 50 parts, among them K1 CQ1-12V, K2 CQ1-12V, K3 CQ1-12V, K4 CQ1-12V, Q1 PN2222, Q2 PN2222, Q3 PN2222, Q4 PN2222, U1 ARDUINO-MEGAFULL

Commit message: update
Parts:
- moved F1 11.4 mm to (31.8, 132.1)
- moved U$2 5.08 mm to (41.9, 113.0)
- moved D2 3.81 mm to (38.1, 64.8)
- moved D4 3.81 mm to (38.1, 29.2)
- moved F/B 3.81 mm to (10.2, 49.5)
- moved F2 3.81 mm to (11.4, 113.0)
- moved K1 3.81 mm to (26.7, 67.3)
- moved K2 3.81 mm to (26.7, 49.5)
- moved K3 3.81 mm to (26.7, 31.8)
- moved LED2 3.81 mm to (49.5, 48.3)
- moved LED3 3.81 mm to (49.5, 29.2)
- moved LED4 3.81 mm to (49.5, 12.7)
- moved OK1 3.81 mm to (44.5, 54.6)
- moved OK2 3.81 mm to (44.5, 72.4)
- moved OK3 3.81 mm to (44.5, 36.8)
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Connections:
- removed net INT: CAN-BUS.7, U1.20
- removed net N$23: F1.2, U$2.IN+
- net VIN: now also F1.2, U$2.IN+
Routing:
- net VIN: track 0.00 -> 186.5 mm, vias 0 -> 3
- net N$23: track 34.3 -> 0.00 mm
- net VCC: track 1422.4 -> 1448.2 mm
- net N$9: track 22.8 -> 45.7 mm
- net N$5: track 22.8 -> 45.7 mm
- net N$24: track 24.5 -> 13.7 mm
- net N$26: track 21.5 -> 28.3 mm
- net GND: track 1435.5 -> 1429.5 mm
- net VINS: track 129.1 -> 132.6 mm
- net N$25: track 9.07 -> 9.92 mm
- net IN4: track 51.6 -> 52.4 mm
Other:
- board size 210.8 x 146.1 mm -> 208.3 x 141 mm

Commit message: update
Routing:
- net VCC: track 1448.2 -> 716.0 mm
- net GND: track 1429.5 -> 1056.0 mm

Commit message: update
Parts:
- moved LED4 1.27 mm to (49.5, 11.4)
Routing:
- net GND: track 1056.0 -> 874.2 mm, vias 10 -> 9
- net D8PWM: track 115.6 -> 162.6 mm
- net VCC: track 716.0 -> 750.4 mm
- net VINS: track 132.6 -> 164.9 mm, vias 2 -> 1
- net D6PWM: track 122.7 -> 106.7 mm, vias 0 -> 3
- net D10PWM: track 73.9 -> 82.5 mm
- net VIN: track 186.5 -> 193.6 mm
- net D7PWM: track 119.3 -> 113.7 mm, vias 0 -> 2
- net !CS: track 60.5 -> 64.6 mm
- net MOSI: track 55.9 -> 59.2 mm
- net LEDS: track 10.5 -> 12.5 mm
- net N$24: track 13.7 -> 15.3 mm
- net LEDS1: track 11.0 -> 12.5 mm
- net INSS1: track 17.3 -> 18.8 mm
- net INS: track 16.8 -> 18.3 mm
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
Commit message: update
Parts:
- moved SENBREAK 12.7 mm to (10.2, 81.3)
- moved R4 9.25 mm to (20.3, 85.1)
- moved R12 2.84 mm to (96.5, 21.6)
- moved R13 2.84 mm to (99.1, 21.6)
- moved CAN-BUS 2.54 mm to (76.2, 11.3)
- moved Q3 2.54 mm to (43.2, 29.2), turned to 0 degrees
- moved R6 2.54 mm to (53.3, 48.3)
- moved R8 2.54 mm to (53.3, 66.0)
- moved U$1 1.80 mm to (92.7, 24.1)
- moved LED1 1.27 mm to (49.5, 64.8)
- moved Q1 1.27 mm to (43.2, 47.0), turned to 0 degrees
- moved R1 1.27 mm to (55.9, 38.1)
- moved R10 1.27 mm to (53.3, 12.7)
- moved Q4 1.27 mm to (43.2, 11.4), turned to 0 degrees
- moved R2 1.27 mm to (53.3, 30.5)
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Routing:
- net GND: track 874.2 -> 588.6 mm, vias 9 -> 13
- net VIN: track 193.6 -> 289.3 mm
- net D8PWM: track 162.6 -> 110.1 mm
- net VCC: track 750.4 -> 791.3 mm, vias 0 -> 2
- net N$26: track 28.3 -> 56.2 mm
- net D13PWM: track 56.8 -> 81.2 mm
- net N$24: track 15.3 -> 27.9 mm
- net D10PWM: track 82.5 -> 69.9 mm
- net D7PWM: track 113.7 -> 103.6 mm
- net MISO: track 47.9 -> 38.9 mm, vias 2 -> 3
- net D11PWM: track 77.1 -> 71.0 mm
- net !SHDN: track 12.5 -> 8.67 mm
- net D9PWM: track 75.4 -> 71.7 mm
- net N$12: track 10.5 -> 14.0 mm
- net N$20: track 10.5 -> 14.0 mm
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- added copper zone on layer 16, net B

Commit message: update
Connections:
- removed net D7: R13.P$1, U$1.8
- new net D48: R13.P$1, U$1.8, U1.48
Routing:
- net D7: track 9.42 -> 0.00 mm
- net D48: track 0.00 -> 9.42 mm
Changed lines of the file:
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@@
 <drawing>
 <settings>
-<setting alwaysvectorfont="no"/>
+<setting alwaysvectorfont="yes"/>
 <setting verticaltext="up"/>
 </settings>
 <grid distance="50" unitdist="mil" unit="mil" style="lines" multiple="1" display="yes" altdistance="5" altunitdist="mil" altunit="mil"/>
 <layers>
-<layer number="1" name="Top" color="4" fill="1" visible="no" active="yes"/>
+<layer number="1" name="Top" color="4" fill="1" visible="yes" active="yes"/>
 <layer number="2" name="Route2" color="16" fill="1" visible="no" active="no"/>
 <layer number="3" name="Route3" color="17" fill="1" visible="no" active="no"/>
@@
 <layer number="19" name="Unrouted" color="6" fill="1" visible="yes" active="yes"/>
 <layer number="20" name="Dimension" color="24" fill="1" visible="yes" active="yes"/>
-<layer number="21" name="tPlace" color="7" fill="1" visible="no" active="yes"/>
-<layer number="22" name="bPlace" color="7" fill="1" visible="no" active="yes"/>
-<layer number="23" name="tOrigins" color="15" fill="1" visible="no" active="yes"/>
-<layer number="24" name="bOrigins" color="15" fill="1" visible="no" active="yes"/>
-<layer number="25" name="tNames" color="7" fill="1" visible="no" active="yes"/>
-<layer number="26" name="bNames" color="7" fill="1" visible="no" active="yes"/>
+<layer number="21" name="tPlace" color="7" fill="1" visible="yes" active="yes"/>
+<layer number="22" name="bPlace" color="7" fill="1" visible="yes" active="yes"/>
+<layer number="23" name="tOrigins" color="15" fill="1" visible="yes" active="yes"/>
+<layer number="24" name="bOrigins" color="15" fill="1" visible="yes" active="yes"/>
+<layer number="25" name="tNames" color="7" fill="1" visible="yes" active="yes"/>
+<layer number="26" name="bNames" color="7" fill="1" visible="yes" active="yes"/>
 <layer number="27" name="tValues" color="7" fill="1" visible="no" active="yes"/>
 <layer number="28" name="bValues" color="7" fill="1" visible="no" active="yes"/>
@@
 <layer number="37" name="tTest" color="7" fill="1" visible="no" active="yes"/>
 <layer number="38" name="bTest" color="7" fill="1" visible="no" active="yes"/>
-<layer number="39" name="tKeepout" color="4" fill="11" visible="no" active="yes"/>
+<layer number="39" name="tKeepout" color="4" fill="11" visible="yes" active="yes"/>
 <layer number="40" name="bKeepout" color="1" fill="11" visible="yes" active="yes"/>
-<layer number="41" name="tRestrict" color="4" fill="10" visible="no" active="yes"/>
+<layer number="41" name="tRestrict" color="4" fill="10" visible="yes" active="yes"/>
 <layer number="42" name="bRestrict" color="1" fill="10" visible="yes" active="yes"/>
 <layer number="43" name="vRestrict" color="2" fill="10" visible="no" active="yes"/>
@@
 <layer number="49" name="Reference" color="7" fill="1" visible="no" active="yes"/>
 <layer number="50" name="dxf" color="7" fill="1" visible="no" active="no"/>
-<layer number="51" name="tDocu" color="7" fill="1" visible="no" active="yes"/>
+<layer number="51" name="tDocu" color="7" fill="1" visible="yes" active="yes"/>
 <layer number="52" name="bDocu" color="7" fill="1" visible="yes" active="yes"/>
 <layer number="53" name="tGND_GNDA" color="7" fill="9" visible="no" active="no"/>
@@
 <wire x1="109.22" y1="27.94" x2="109.22" y2="13.97" width="1.27" layer="16"/>
 </signal>
-<signal name="D7">
-<contactref element="U$1" pad="8"/>
-<contactref element="R13" pad="P$1"/>
-<wire x1="95.25" y1="24.13" x2="96.52" y2="22.86" width="1.27" layer="16"/>
-<wire x1="99.06" y1="25.4" x2="99.06" y2="22.86" width="1.27" layer="16"/>
-<wire x1="99.06" y1="22.86" x2="96.52" y2="22.86" width="1.27" layer="16"/>
-<wire x1="92.71" y1="24.13" x2="95.25" y2="24.13" width="1.27" layer="16"/>
-</signal>
 <signal name="!SHDN">
 <contactref element="U$1" pad="9"/>
@@
 </polygon>
 </signal>
+<signal name="D48">
+<contactref element="U1" pad="48"/>
+<contactref element="U$1" pad="8"/>
+<contactref element="R13" pad="P$1"/>
+<wire x1="95.25" y1="24.13" x2="96.52" y2="22.86" width="1.27" layer="16"/>
+<wire x1="99.06" y1="25.4" x2="99.06" y2="22.86" width="1.27" layer="16"/>
+<wire x1="99.06" y1="22.86" x2="96.52" y2="22.86" width="1.27" layer="16"/>
+<wire x1="92.71" y1="24.13" x2="95.25" y2="24.13" width="1.27" layer="16"/>
+<wire x1="99.06" y1="25.4" x2="102.87" y2="31.75" width="0" layer="19" extent="1-1"/>
+</signal>
 </signals>
