File: MB_AutoCar/main.sch (EAGLE design)
At the start: 48 parts, among them J2 Out1, J4 Out2, K1 CQ1-12V, K2 CQ1-12V, K3 CQ1-12V, K4 CQ1-12V, Q1 PN2222, Q2 PN2222, Q3 PN2222, Q4 PN2222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

Commit message: update
Parts:
- removed PWMS: Out1, SparkFun-Connectors:M02PTH3
- added ENCODER: (no value), SparkFun-Connectors:CONN_15
- added PWMS1: Out1, SparkFun-Connectors:M02PTH3
- added U$3, U$4: (no value), TLP250:TLP250V1
- renumbered ON/OFF to SPEED, SPEEDS to ON/OFFS
Connections:
- removed net N$13: K42.S, SPEED-1.KL
- removed net PWMS: ON/OFFS-1.KL, PWMS.1
- new net D22: ENCODER.1, U1.22
- new net D24: ENCODER.2, U1.24
- new net D26: ENCODER.3, U1.26
- new net D28: ENCODER.4, U1.28
- new net D30: ENCODER.5, U1.30
- new net D32: ENCODER.6, U1.32
- new net D34: ENCODER.7, U1.34
- new net D36: ENCODER.8, U1.36
- new net D38: ENCODER.9, U1.38
- new net D40: ENCODER.10, U1.40
- new net D42: ENCODER.11, U1.42
- new net D44: ENCODER.12, U1.44
- new net D46: ENCODER.13, U1.46
- new net N$1: PWMS1.1, SPEED-1.KL
- new net N$2: K12.S, ON/OFFS-1.KL
- new net VIN: ENCODER.14
- net D12PWM: now also K42.S, PWMS1.2
- net D13PWM: no longer K12.S, PWMS.2
- net GND: now also ENCODER.15
- net IN1: now also U1.5; no longer U1.2
- net IN2: now also U1.4; no longer U1.3
- net IN3: now also U1.3; no longer U1.4
- net IN4: now also U1.2; no longer U1.5
Other:
- moved on the sheet: U1
