File: MB_AutoCar/main.sch (EAGLE design)
At the start: 50 parts, among them K1 CQ1-12V, K2 CQ1-12V, K3 CQ1-12V, K4 CQ1-12V, Q1 PN2222, Q2 PN2222, Q3 PN2222, Q4 PN2222, U1 ARDUINO-MEGAFULL

Commit message: update
Connections:
- removed net INT: CAN-BUS.7, U1.20(SDA)
- removed net N$23: F1.2, U$2.IN+
- net VIN: now also F1.2, U$2.IN+
Changed lines of the file:
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@@
 </classes>
 <parts>
-<part name="U$2" library="diy-modules" deviceset="DC-DC-STEP-DOWN-LM2596" device=""/>
 <part name="OK1" library="optocoupler" library_urn="urn:adsk.eagle:library:320" deviceset="PC817" device="" package3d_urn="urn:adsk.eagle:package:21938/1"/>
 <part name="Q1" library="transistor-npn" library_urn="urn:adsk.eagle:library:398" deviceset="BC447*" device="" package3d_urn="urn:adsk.eagle:package:28989/2" value="PN2222"/>
@@
 <part name="PWMS2" library="SparkFun-Connectors" deviceset="M02" device="PTH3" value="Out1"/>
 <part name="U1" library="SparkFun-Boards" deviceset="ARDUINO-MEGA" device="FULL"/>
+<part name="U$2" library="diy-modules" deviceset="DC-DC-STEP-DOWN-LM2596" device=""/>
 </parts>
 <sheets>
@@
 </plain>
 <instances>
-<instance part="U$2" gate="G$1" x="88.9" y="12.7" smashed="yes">
-<attribute name="NAME" x="76.2" y="27.94" size="1.778" layer="95"/>
-<attribute name="VALUE" x="76.2" y="25.4" size="1.778" layer="96"/>
-</instance>
 <instance part="OK1" gate="A" x="53.34" y="147.32" smashed="yes">
 <attribute name="NAME" x="46.355" y="153.035" size="1.778" layer="95"/>
@@
 <attribute name="NAME" x="165.1" y="115.062" size="1.778" layer="95"/>
 <attribute name="VALUE" x="165.1" y="5.08" size="1.778" layer="96"/>
+</instance>
+<instance part="U$2" gate="G$1" x="88.9" y="12.7" smashed="yes">
+<attribute name="NAME" x="76.2" y="27.94" size="1.778" layer="95"/>
+<attribute name="VALUE" x="76.2" y="25.4" size="1.778" layer="96"/>
 </instance>
 </instances>
@@
 </segment>
 <segment>
-<pinref part="U$2" gate="G$1" pin="OUT-"/>
 <wire x1="106.68" y1="7.62" x2="114.3" y2="7.62" width="0.1524" layer="91"/>
 <pinref part="GND3" gate="1" pin="GND"/>
+<pinref part="U$2" gate="G$1" pin="OUT-"/>
 </segment>
 <segment>
@@
 </segment>
 </net>
-<net name="INT" class="0">
-<segment>
-<pinref part="CAN-BUS" gate="G$1" pin="7"/>
-<wire x1="88.9" y1="114.3" x2="91.44" y2="114.3" width="0.1524" layer="91"/>
-<label x="91.44" y="114.3" size="1.778" layer="95"/>
-</segment>
-<segment>
-<wire x1="200.66" y1="93.98" x2="203.2" y2="93.98" width="0.1524" layer="91"/>
-<label x="203.2" y="93.98" size="1.778" layer="95"/>
-<pinref part="U1" gate="G$1" pin="20(SDA)"/>
-</segment>
-</net>
 <net name="MISO" class="0">
 <segment>
@@
 </segment>
 <segment>
-<pinref part="U$2" gate="G$1" pin="OUT+"/>
 <wire x1="106.68" y1="17.78" x2="114.3" y2="17.78" width="0.1524" layer="91"/>
 <label x="114.3" y="17.78" size="1.778" layer="95"/>
-</segment>
-</net>
-<net name="N$23" class="0">
-<segment>
-<pinref part="U$2" gate="G$1" pin="IN+"/>
-<pinref part="F1" gate="G$1" pin="2"/>
-<wire x1="68.58" y1="17.78" x2="71.12" y2="17.78" width="0.1524" layer="91"/>
+<pinref part="U$2" gate="G$1" pin="OUT+"/>
 </segment>
 </net>
@@
 <net name="N$25" class="0">
 <segment>
-<pinref part="U$2" gate="G$1" pin="IN-"/>
 <pinref part="F2" gate="G$1" pin="2"/>
 <wire x1="68.58" y1="7.62" x2="71.12" y2="7.62" width="0.1524" layer="91"/>
+<pinref part="U$2" gate="G$1" pin="IN-"/>
 </segment>
 </net>
@@
 <label x="99.06" y="48.26" size="1.778" layer="95"/>
 </segment>
-</net>
+<segment>
+<pinref part="F1" gate="G$1" pin="2"/>
+<wire x1="68.58" y1="17.78" x2="71.12" y2="17.78" width="0.1524" layer="91"/>
+<pinref part="U$2" gate="G$1" pin="IN+"/>
+<label x="71.12" y="20.32" size="1.778" layer="95"/>
+<wire x1="71.12" y1="17.78" x2="71.12" y2="20.32" width="0.1524" layer="91"/>
+<junction x="71.12" y="17.78"/>
+</segment>
+</net>

Commit message: update
Connections:
- removed net D7: R13.1, U$1.~LDAC
- new net D48: R13.1, U$1.~LDAC, U1.48
Changed lines of the file:
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@@
-</segment>
-</net>
-<net name="D7" class="0">
-<segment>
-<pinref part="U$1" gate="A" pin="~LDAC"/>
-<wire x1="30.48" y1="55.88" x2="17.78" y2="55.88" width="0.1524" layer="91"/>
-<pinref part="R13" gate="G$1" pin="1"/>
-<wire x1="17.78" y1="60.96" x2="17.78" y2="55.88" width="0.1524" layer="91"/>
-<label x="25.4" y="55.88" size="1.778" layer="95"/>
 </segment>
 </net>
@@
 </segment>
 </net>
+<net name="D48" class="0">
+<segment>
+<pinref part="U1" gate="G$1" pin="48"/>
+<wire x1="200.66" y1="22.86" x2="203.2" y2="22.86" width="0.1524" layer="91"/>
+<label x="203.2" y="22.86" size="1.778" layer="95"/>
+</segment>
+<segment>
+<pinref part="U$1" gate="A" pin="~LDAC"/>
+<wire x1="30.48" y1="55.88" x2="17.78" y2="55.88" width="0.1524" layer="91"/>
+<pinref part="R13" gate="G$1" pin="1"/>
+<wire x1="17.78" y1="60.96" x2="17.78" y2="55.88" width="0.1524" layer="91"/>
+<label x="25.4" y="55.88" size="1.778" layer="95"/>
+</segment>
+</net>
