File: MB_AutoCarV2/main.sch (EAGLE design)
At the start: 44 parts, among them K1 CQ1-12V, K2 CQ1-12V, K3 CQ1-12V, K4 CQ1-12V, Q1 PN2222, Q2 PN2222, Q3 PN2222, Q4 PN2222, U1 ARDUINO-MEGAFULL

Commit message: update
Parts:
- removed ENCODER: (no value), SparkFun-Connectors:CONN_15
- added ENCODER1: (no value), SparkFun-Connectors:CONN_15
- renumbered D1 to D22, D2 to D11, D4 to D33, D5 to D44
Connections:
- removed net D22: ENCODER.1, U1.22
- removed net D24: ENCODER.2, U1.24
- removed net D26: ENCODER.3, U1.26
- removed net D28: ENCODER.4, U1.28
- removed net D30: ENCODER.5, U1.30
- removed net D32: ENCODER.6, U1.32
- removed net D34: ENCODER.7, U1.34
- removed net D36: ENCODER.8, U1.36
- removed net D38: ENCODER.9, U1.38
- removed net D40: ENCODER.10, U1.40
- removed net D42: ENCODER.11, U1.42
- removed net D44: ENCODER.12, U1.44
- removed net D46: ENCODER.13, U1.46
- removed net D48: U1.48
- removed net N$1: K42.S, SPEED-1.KL
- new net D23: ENCODER1.2, U1.23
- new net D25: ENCODER1.3, U1.25
- new net D27: ENCODER1.4, U1.27
- new net D29: ENCODER1.5, U1.29
- new net D31: ENCODER1.6, U1.31
- new net D33: ENCODER1.7, U1.33
- new net D35: ENCODER1.8, U1.35
- new net D37: ENCODER1.9, U1.37
- new net D39: ENCODER1.10, U1.39
- new net D41: ENCODER1.11, U1.41
- new net D43: ENCODER1.12, U1.43
- new net D45: ENCODER1.13, U1.45
- new net D47: ENCODER1.14, U1.47
- new net D49: U1.49
- new net N$13: K42.O, SPEED-3.KL
- net !CS: now also CAN-BUS.5; no longer CAN-BUS.3
- net 22: now also Q1.C; no longer Q2.C
- net D12PWM: now also K42.S, SPEED-1.KL; no longer K42.O, SPEED-3.KL
- net GND: now also ENCODER1.15; no longer ENCODER.15, U1.GND@0, U1.GND@1
- net GND-: now also Q2.C; no longer Q1.C
- net INS: now also OK2.A; no longer OK1.A
- net INSS: now also OK1.A; no longer OK2.A
- net LED: now also OK2.C; no longer OK1.C
- net LEDS: now also OK1.C; no longer OK2.C
- net MISO: now also CAN-BUS.3; no longer CAN-BUS.5
- net N$12: now also Q2.B; no longer Q1.B
- net N$20: now also Q1.B; no longer Q2.B
- net N$22: now also OK1.EMIT; no longer OK2.EMIT
- net OTP: now also OK2.EMIT; no longer OK1.EMIT
- net VCC: no longer U1.5V@0
- net VIN: now also ENCODER1.1; no longer ENCODER.14
Other:
- moved on the sheet: OK1, OK2, Q1, Q2

Commit message: update
Changed lines of the file:
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@@
 <wire x1="129.54" y1="22.86" x2="129.54" y2="20.32" width="0.1524" layer="91"/>
 <pinref part="GND11" gate="1" pin="GND"/>
-</segment>
-<segment>
+<wire x1="129.54" y1="22.86" x2="111.76" y2="22.86" width="0.1524" layer="91"/>
+<junction x="129.54" y="22.86"/>
+<wire x1="111.76" y1="22.86" x2="111.76" y2="12.7" width="0.1524" layer="91"/>
+<wire x1="111.76" y1="12.7" x2="88.9" y2="12.7" width="0.1524" layer="91"/>
+<wire x1="88.9" y1="12.7" x2="88.9" y2="20.32" width="0.1524" layer="91"/>
 <pinref part="ENCODER1" gate="G$1" pin="15"/>
-<wire x1="93.98" y1="20.32" x2="91.44" y2="20.32" width="0.1524" layer="91"/>
-<label x="88.9" y="20.32" size="1.778" layer="95"/>
+<wire x1="88.9" y1="20.32" x2="93.98" y2="20.32" width="0.1524" layer="91"/>
 </segment>
 </net>

Commit message: update
Connections:
- removed net IN2: R3.1, U1.4
- net IN1: now also R3.1
Changed lines of the file:
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@@
 <pinref part="U1" gate="G$1" pin="5"/>
 </segment>
-</net>
-<net name="IN2" class="0">
 <segment>
 <pinref part="R3" gate="G$1" pin="1"/>
@@
 <label x="2.54" y="157.48" size="1.778" layer="95"/>
 </segment>
-<segment>
-<wire x1="137.16" y1="50.8" x2="132.08" y2="50.8" width="0.1524" layer="91"/>
-<label x="132.08" y="50.8" size="1.778" layer="95"/>
-<pinref part="U1" gate="G$1" pin="4"/>
-</segment>
 </net>
