File: ESP32-UC20G/ModbusGateway4GWiFi.brd (EAGLE design)
At the start: 92.1 x 87 mm, 84 parts, among them IC1 DALC208SC6, J1 67910-0002, J3 TxRx, J4 I2C, U2 ESP-WROOM-32, X1 SIMLOCK-C707_10M006_512_2, X3 Sense

Commit message: update
Parts:
- removed C10, C4: 0.1uF, SparkFun-Passives:0805
- removed C2: 0.1, SparkFun-Passives:0805
- removed C3: 1000/10, adafruit:140CLH-1010
- removed F1: (no value), fuse:SH22,5A
- removed J4: I2C, SparkFun-Connectors:MOLEX-1X4
- removed JP1: RT, SparkFun:1X02
- removed JP4: Bypass GND, SparkFun-Retired:SJ_2S-NO
- removed JP5: Bypass VCC, SparkFun-Retired:SJ_2S-NO
- removed LED13: IN1, adafruit:CHIP-LED0805
- removed LED14: IN2, adafruit:CHIP-LED0805
- removed LED2: PW, led:CHIP-LED0805
- removed OK7, OK8: PC817, optocoupler:DIL4-SMD
- removed R10, R20, R24, R36, R38: 10k, SparkFun-Resistors:0805
- removed R12: 56k, SparkFun-Resistors:0805
- removed R2: 1k, SparkFun-Resistors:0805
- removed R37, R39: 2.2k, SparkFun-Resistors:0805
- removed SJ3: JUMP COM to GND, SparkFun:SJ_2S-NO
- removed U$15, U$16, U$17, U$18: (no value), holes:3,2
- removed U$2: 220VAC/12VDC, ES-CONNECTOR:5EHDRC-2P
- removed U$3: In12, ES-CONNECTOR:5EHDRC-2P
- removed U$4: MAX13487, TCS-MAXIM:SOIC8-1.27-5X4MM
- removed U$5: Com, ES-CONNECTOR:5EHDRC-2P
- removed U$6: DC LM2596 5V, diy-modules:DC-DC-STEP-DOWN-LM2596
- removed U$8: RS485, ES-CONNECTOR:5EHDRC-2P
- removed X3: Sense, Rembrandt Electronics - JST XH Connectors v1-0:JST-XH-04-PACKAGE-LONG-PAD
- added LED1: PW, led:CHIP-LED0805
- LED4: value R_RX -> RRX
- LED5: value R_TX -> RTX
- LED8: value A_L -> STAT
- R1: value 120 -> 4.7k
- R5: value 56k -> 1k
- U$1: value HIECUBE -> 220VAC/12VDC; device HICUBE:HIECUBE -> ES-CONNECTOR:5EHDRC-2P
- moved R4 177.9 mm to (-86.4, 109.2), turned to 0 degrees
- moved R3 172.7 mm to (-82.5, 109.2), turned to 0 degrees
- moved JP16 166.7 mm to (-38.1, 118.1)
- moved C17 165.0 mm to (-87.6, 115.6), turned to 0 degrees
- moved JP10 161.2 mm to (-30.5, 118.1), flipped to the top
- moved LED3 160.0 mm to (-40.6, 109.2), turned to 0 degrees
- moved C14 155.8 mm to (-86.4, 88.9), turned to 0 degrees
- moved IC1 155.1 mm to (-69.8, 109.2), turned to 0 degrees
- moved C1 153.5 mm to (-61.0, 115.6), turned to 0 degrees
- moved C13 150.9 mm to (-83.8, 115.6), turned to 0 degrees
- moved C7 148.3 mm to (-72.4, 115.6), turned to 0 degrees
- moved R7 147.7 mm to (-22.9, 115.6)
- moved C5 143.4 mm to (-64.8, 115.6), turned to 0 degrees
- moved C12 142.5 mm to (-80.0, 115.6), turned to 0 degrees
- moved S4 141.2 mm to (-77.5, 88.9), turned to 0 degrees
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Connections:
- removed net A(+): R1.1, R5.2, U$4.6, U$8.P$2
- removed net B(-): JP1.1, R12.1, U$4.7, U$8.P$1
- removed net COM: LED13.C, LED14.C, SJ3.2, U$5.P$1
- removed net N$26: F1.2, U$1.P$1
- removed net N$5: JP4.1, U$1.P$2, U$2.P$1, U$6.IN-
- removed net N$6: LED2.A, R2.1
- removed net N$60: OK7.1, R37.1
- removed net N$62: LED13.A, OK7.2
- removed net N$63: OK8.1, R39.1
- removed net N$65: LED14.A, OK8.2
- removed net N$68: R37.2, U$3.P$2
- removed net N$71: R39.2, U$3.P$1
- removed net SCL: J4.4, R20.1, U2.36
- removed net SDA: J4.3, R24.1, U2.33
- removed net VS: F1.1, JP5.1, U$2.P$2, U$6.IN+
- new net GPIO21_RSET: J1.22, R1.2, U2.33
- new net N$2: C6.1, U$1.P$2, U$7.IN+
- net 3.3V: now also R1.1, R5.2; no longer R10.2, R20.2, R24.2, R36.1, R38.1
- net GND: now also LED1.C, U$1.P$1; no longer C10.2, C2.2, C3.-, C4.2, J4.1, JP4.2, LED2.C, OK7.3, OK8.3, R12.2, SJ3.1, U$1.P$5, U$4.5, U$6.OUT-, X3.1
- net GPIO25: no longer OK7.4, R36.2
- net GPIO26: no longer OK8.4, R38.2
- net GPIO32: no longer C4.1, R10.1, X3.4
- net GPIO33: no longer X3.3
- net N$1: now also LED1.A, R5.1; no longer JP1.2, R1.2
- net RX2: no longer U$4.1
- net TX2: no longer U$4.4
- net VCC: no longer C10.1, C2.1, C3.+, C6.1, J4.2, JP5.2, R2.2, R5.1, U$1.P$3, U$4.2, U$4.3, U$4.8, U$5.P$2, U$6.OUT+, U$7.IN+, X3.2
Routing:
- net GND: track 609.2 -> 0.00 mm, vias 21 -> 0
- net 3.3V: track 373.7 -> 0.00 mm, vias 12 -> 0
- net VCC: track 251.8 -> 0.00 mm, vias 2 -> 0
- net GPIO4: track 70.5 -> 0.00 mm, vias 2 -> 0
- net RX2: track 63.0 -> 0.00 mm, vias 3 -> 0
- net TX2: track 59.0 -> 0.00 mm, vias 3 -> 0
- net GPIO33: track 58.8 -> 0.00 mm, vias 1 -> 0
- net S_RST: track 50.5 -> 0.00 mm, vias 2 -> 0
- net VS: track 49.8 -> 0.00 mm
- net GPIO32: track 45.2 -> 0.00 mm
- net S_VSIM: track 44.7 -> 0.00 mm
- net A(+): track 44.3 -> 0.00 mm
- net COM: track 43.2 -> 0.00 mm, vias 2 -> 0
- net S_DATA: track 42.8 -> 0.00 mm
- net N$5: track 41.9 -> 0.00 mm
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- removed copper zone on layer 1, net GND
- removed copper zone on layer 16, net GND
Other:
- board size 92.1 x 87 mm -> 160 x 100 mm
- board text removed: "A - B"
- board text removed: "C NO"
- board text removed: "L - N"
